File: control_board_Kicad/KiCad-Pi-Pico/KiCad-Pi-Pico.kicad_pcb (KiCad board)
At the start: 2 copper layers, 0 parts

Commit message: KiCad update
Parts:
- added J1: DB25_Plug_MountingHoles, Connector_Dsub:DSUB-25_Male_Horizontal_P2.77x2.84mm_EdgePinOffset4.94mm_Housed_MountingHolesOffset7.48mm, F.Cu at (105.5, 83.4)
- added Q1: 2N7002, Package_TO_SOT_SMD:SOT-23, F.Cu at (175.0, 75.0)
- added Q2: 2N7002, Package_TO_SOT_SMD:SOT-23, F.Cu at (160.0, 75.0)
- added Q3: 2N7002, Package_TO_SOT_SMD:SOT-23, F.Cu at (145.0, 75.0)
- added Q4: 2N7002, Package_TO_SOT_SMD:SOT-23, F.Cu at (130.0, 75.0)
- added R1: 4.7 kΩ, Resistor_SMD:R_1206_3216Metric_Pad1.30x1.75mm_HandSolder, F.Cu at (180.0, 75.0)
- added R10: 4.7 kΩ, Resistor_SMD:R_1206_3216Metric_Pad1.30x1.75mm_HandSolder, F.Cu at (115.0, 120.0)
- added R11: 4.7 kΩ, Resistor_SMD:R_1206_3216Metric_Pad1.30x1.75mm_HandSolder, F.Cu at (115.0, 115.0)
- added R12: 4.7 kΩ, Resistor_SMD:R_1206_3216Metric_Pad1.30x1.75mm_HandSolder, F.Cu at (115.0, 110.0)
- added R13: 4.7 kΩ, Resistor_SMD:R_1206_3216Metric_Pad1.30x1.75mm_HandSolder, F.Cu at (115.0, 105.0)
- added R14: 4.7 kΩ, Resistor_SMD:R_1206_3216Metric_Pad1.30x1.75mm_HandSolder, F.Cu at (115.0, 95.0)
- added R2: 4.7 kΩ, Resistor_SMD:R_1206_3216Metric_Pad1.30x1.75mm_HandSolder, F.Cu at (165.0, 75.0)
- added R3: 4.7 kΩ, Resistor_SMD:R_1206_3216Metric_Pad1.30x1.75mm_HandSolder, F.Cu at (150.0, 75.0)
- added R4: 4.7 kΩ, Resistor_SMD:R_1206_3216Metric_Pad1.30x1.75mm_HandSolder, F.Cu at (172.5, 80.0)
- added R5: 4.7 kΩ, Resistor_SMD:R_1206_3216Metric_Pad1.30x1.75mm_HandSolder, F.Cu at (157.5, 80.0)
- added R6: 4.7 kΩ, Resistor_SMD:R_1206_3216Metric_Pad1.30x1.75mm_HandSolder, F.Cu at (142.5, 80.0)
- added R7: 4.7 kΩ, Resistor_SMD:R_1206_3216Metric_Pad1.30x1.75mm_HandSolder, F.Cu at (115.0, 100.0)
- added R8: 4.7 kΩ, Resistor_SMD:R_1206_3216Metric_Pad1.30x1.75mm_HandSolder, F.Cu at (127.5, 80.0)
- added R9: 4.7 kΩ, Resistor_SMD:R_1206_3216Metric_Pad1.30x1.75mm_HandSolder, F.Cu at (135.0, 75.0)
- added RV1: R_Potentiometer_US, Potentiometer_THT:Potentiometer_Bourns_3386W_Horizontal, F.Cu at (170.0, 127.5)
- added RV2: R_Potentiometer_US, Potentiometer_THT:Potentiometer_Bourns_3386W_Horizontal, F.Cu at (159.9, 122.5)
- added SW1: SW_Push, Button_Switch_SMD:SW_Tactile_SPST_NO_Straight_CK_PTS636Sx25SMTRLFS, F.Cu at (185.0, 120.0)
- added U1: SC0915, SC0915:MODULE_SC0915, F.Cu at (150.0, 100.0)
- added U2: AD5761RBRUZ, AD5761RBRUZ:SOP65P640X120-16N, F.Cu at (150.0, 125.0)
- added U3: LM285D-2.5, Package_SO:SOIC-8_3.9x4.9mm_P1.27mm, F.Cu at (140.0, 125.0)
Routing:
- net GND: track 0.00 -> 105.4 mm, vias 0 -> 3
- net +2V5REF: track 0.00 -> 40.4 mm, vias 0 -> 2
- net Net-(J1-P23): track 0.00 -> 15.0 mm
- net Net-(J1-P24): track 0.00 -> 14.9 mm
- net Net-(J1-P19): track 0.00 -> 14.5 mm
- net Net-(U1-GP9): track 0.00 -> 12.0 mm
- net Net-(U1-GP3): track 0.00 -> 12.0 mm
- added copper zone on F.Cu, net +5V
- added copper zone on B.Cu, net GND
Other:
- board outline added: 100 x 70 mm
