File: control_board_Kicad/KiCad-Pi-Pico/KiCad-Pi-Pico.kicad_pcb (KiCad board)
At the start: 2 copper layers, 100 x 70 mm, 25 parts, among them J1 DB25_Plug_MountingHoles, Q1 2N7002, Q2 2N7002, Q3 2N7002, Q4 2N7002, SW1 SW_Push, U1 SC0915, U2 AD5761RBRUZ, U3 LM285D-2.5

Commit message: update
Routing:
- net GND: track 105.4 -> 97.3 mm
- net Net-(Q4-D): track 0.00 -> 5.01 mm
- net Net-(J1-P20): track 0.00 -> 5.01 mm
- net Net-(J1-P16): track 0.00 -> 5.01 mm
- net Net-(J1-P15): track 0.00 -> 5.01 mm
- net Net-(Q4-G): track 0.00 -> 4.31 mm
- net Net-(Q3-G): track 0.00 -> 4.31 mm
- net Net-(Q2-G): track 0.00 -> 4.31 mm
- net Net-(Q1-G): track 0.00 -> 4.31 mm
Changed lines of the file:
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@@
-	)
-	(segment
-		(start 147.05 73.45)
-		(end 150 73.45)
-		(width 0.2)
-		(layer "F.Cu")
-		(net 1)
 	)
 	(segment
@@
 	)
 	(segment
-		(start 160.9375 74.05)
-		(end 164.4 74.05)
-		(width 0.2)
-		(layer "F.Cu")
-		(net 1)
-	)
-	(segment
 		(start 175.3375 73.45)
 		(end 175.9375 74.05)
@@
 	)
 	(segment
-		(start 146.45 74.05)
-		(end 147.05 73.45)
-		(width 0.2)
-		(layer "F.Cu")
-		(net 1)
-	)
-	(segment
 		(start 151 124.5)
 		(end 150.975 124.475)
@@
 		(start 145.3375 73.45)
 		(end 145.9375 74.05)
-		(width 0.2)
-		(layer "F.Cu")
-		(net 1)
-	)
-	(segment
-		(start 164.4 74.05)
-		(end 165 73.45)
 		(width 0.2)
 		(layer "F.Cu")
@@
 	)
 	(segment
+		(start 129.05 75.0125)
+		(end 129.0625 75)
+		(width 0.2)
+		(layer "F.Cu")
+		(net 2)
+	)
+	(segment
+		(start 129.05 80)
+		(end 129.05 75.0125)
+		(width 0.2)
+		(layer "F.Cu")
+		(net 2)
+	)
+	(segment
 		(start 114.315 102.765)
 		(end 105.505331 102.765)
@@
 	)
 	(segment
+		(start 174.05 75.0125)
+		(end 174.0625 75)
+		(width 0.2)
+		(layer "F.Cu")
+		(net 9)
+	)
+	(segment
+		(start 174.05 80)
+		(end 174.05 75.0125)
+		(width 0.2)
+		(layer "F.Cu")
+		(net 9)
+	)
+	(segment
+		(start 159.05 75.0125)
+		(end 159.0625 75)
+		(width 0.2)
+		(layer "F.Cu")
+		(net 15)
+	)
+	(segment
+		(start 159.05 80)
+		(end 159.05 75.0125)
+		(width 0.2)
+		(layer "F.Cu")
+		(net 15)
+	)
+	(segment
 		(start 115.375 111.175)
 		(end 107.160966 111.175)
@@
 	)
 	(segment
+		(start 144.05 75.0125)
+		(end 144.0625 75)
+		(width 0.2)
+		(layer "F.Cu")
+		(net 19)
+	)
+	(segment
+		(start 144.05 80)
+		(end 144.05 75.0125)
+		(width 0.2)
+		(layer "F.Cu")
+		(net 19)
+	)
+	(segment
+		(start 179.4 75.95)
+		(end 180 76.55)
+		(width 0.2)
+		(layer "F.Cu")
+		(net 20)
+	)
+	(segment
+		(start 175.9375 75.95)
+		(end 179.4 75.95)
+		(width 0.2)
+		(layer "F.Cu")
+		(net 20)
+	)
+	(segment
+		(start 164.4 75.95)
+		(end 165 76.55)
+		(width 0.2)
+		(layer "F.Cu")
+		(net 21)
+	)
+	(segment
+		(start 160.9375 75.95)
+		(end 164.4 75.95)
+		(width 0.2)
+		(layer "F.Cu")
+		(net 21)
+	)
+	(segment
+		(start 149.4 75.95)
+		(end 150 76.55)
+		(width 0.2)
+		(layer "F.Cu")
+		(net 22)
+	)
+	(segment
+		(start 145.9375 75.95)
+		(end 149.4 75.95)
+		(width 0.2)
+		(layer "F.Cu")
+		(net 22)
+	)
+	(segment
+		(start 134.4 75.95)
+		(end 135 76.55)
+		(width 0.2)
+		(layer "F.Cu")
+		(net 23)
+	)
+	(segment
+		(start 130.9375 75.95)
+		(end 134.4 75.95)
+		(width 0.2)
+		(layer "F.Cu")
+		(net 23)
+	)
+	(segment

Commit message: KiCad updated
Parts:
- U1: footprint SC0915:MODULE_SC0915 -> RPi_Pico:RPi_Pico_SMD_TH
- moved RV2 58.1 mm to (115.8, 84.7)
- moved R14 49.0 mm to (164.0, 95.8), turned to 90 degrees
- moved R13 32.6 mm to (146.2, 95.8), turned to 90 degrees
- moved R7 31.5 mm to (146.2, 104.2), turned to -90 degrees
- moved U2 30.8 mm to (119.3, 122.0)
- moved R12 29.8 mm to (141.2, 95.8), turned to 90 degrees
- moved R11 28.7 mm to (136.2, 95.8), turned to 90 degrees
- moved R10 20.4 mm to (135.2, 122.2), turned to 180 degrees
- moved SW1 14.5 mm to (170.5, 119.2)
- moved RV1 11.2 mm to (162.5, 119.2), turned to 180 degrees
- moved R8 10.6 mm to (138.1, 80.0), turned to 180 degrees
- moved Q4 7.45 mm to (137.4, 75.0)
- moved R9 7.45 mm to (142.4, 75.0)
- moved U3 6.66 mm to (145.5, 121.2), turned to 90 degrees
- moved Q1 6.00 mm to (169.0, 75.0)
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Routing:
- net Net-(U1-GP9): track 12.0 -> 92.7 mm, vias 0 -> 1
- net Net-(J1-P15): track 5.01 -> 81.3 mm, vias 0 -> 2
- net Net-(J1-P20): track 5.01 -> 76.3 mm, vias 0 -> 2
- net Net-(J1-P16): track 5.01 -> 74.7 mm, vias 0 -> 2
- net GND: track 97.3 -> 32.5 mm, vias 3 -> 6
- net Net-(Q4-D): track 5.01 -> 60.3 mm, vias 0 -> 2
- net Net-(U1-GP26): track 0.00 -> 54.5 mm, vias 0 -> 2
- net Net-(U1-GP3): track 12.0 -> 64.6 mm
- net Net-(J1-P24): track 14.9 -> 59.2 mm
- net Net-(J1-P23): track 15.0 -> 56.4 mm
- net Net-(J1-P19): track 14.5 -> 55.5 mm, vias 0 -> 1
- net +2V5REF: track 40.4 -> 0.73 mm, vias 2 -> 0
- net Net-(Q4-G): track 4.31 -> 42.6 mm, vias 0 -> 2
- net Net-(Q2-G): track 4.31 -> 26.6 mm, vias 0 -> 2
- net Net-(Q3-G): track 4.31 -> 19.6 mm
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Other:
- board size 100 x 70 mm -> 85.5 x 60 mm

Commit message: PCB design finished
Parts:
- added U4: PCN2-S5-S12-S, PCN2_S5_S12_S:CONV_PCN2-S5-S12-S, F.Cu at (135.3, 118.1)
- moved U2 44.1 mm to (157.5, 100.0)
- moved U3 19.5 mm to (126.0, 120.0)
- moved R10 17.8 mm to (118.0, 118.0), turned to 0 degrees
Connections:
- J1 pad 0: unconnected-(J1-PAD-Pad0) -> GND
- U2 pad 5: GND -> AGND
- U2 pad 6: GND -> AGND
- U2 pad 8: +10V -> +12V
Routing:
- net Net-(U2-VOUT): track 0.00 -> 72.9 mm, vias 0 -> 3
- net AGND: track 0.00 -> 65.1 mm, vias 0 -> 3
- net +12V: track 0.00 -> 59.5 mm, vias 0 -> 3
- net +2V5REF: track 0.73 -> 52.1 mm, vias 0 -> 2
- net Net-(U1-GP9): track 92.7 -> 51.3 mm
- net Net-(U1-GP12): track 0.00 -> 32.4 mm, vias 0 -> 2
- net Net-(U1-3V3_EN): track 10.4 -> 31.0 mm, vias 0 -> 2
- net Net-(U1-GP26): track 54.5 -> 73.5 mm
- net Net-(U1-GP7): track 0.00 -> 11.4 mm, vias 0 -> 1
- net Net-(U1-GP6): track 0.00 -> 7.14 mm
- net Net-(U1-GP4): track 0.00 -> 6.97 mm
- net Net-(U1-GP5): track 0.00 -> 6.73 mm
- net Net-(J1-P19): track 55.5 -> 54.8 mm
- net Net-(J1-P24): track 59.2 -> 59.9 mm
- net GND: track 32.5 -> 32.2 mm, vias 6 -> 8
Other:
- board size 85.5 x 60 mm -> 83 x 60 mm

Commit message: update PCB design
Parts:
- added C1: 4.7 µF, Capacitor_SMD:C_0402_1005Metric_Pad0.74x0.62mm_HandSolder, F.Cu at (131.6, 96.8)
- added C2: 4.7 µF, Capacitor_SMD:C_0402_1005Metric_Pad0.74x0.62mm_HandSolder, F.Cu at (131.6, 103.2)
- added G***: LOGO, UW-Madison Logo:logo, F.Cu at (116.0, 120.0)
- added G***: LOGO, UW-Madison Logo:logo, B.Cu at (116.0, 120.0)
- added SW2: SW_Push, Button_Switch_SMD:SW_Tactile_SPST_NO_Straight_CK_PTS636Sx25SMTRLFS, F.Cu at (168.6, 119.2)
- added U5: LM285LPR-2-5, LM285LPR_2_5:LP3, F.Cu at (128.8, 120.6)
- U3: value LM285D-2.5 -> LM4132BMF-2.5; footprint Package_SO:SOIC-8_3.9x4.9mm_P1.27mm -> LM4132BMF_2_5_NOPB:DBV0005A_M
- moved U3 43.9 mm to (166.0, 102.0), turned to 180 degrees
- moved R10 24.9 mm to (138.0, 103.2), turned to 180 degrees
- moved SW1 4.10 mm to (174.6, 119.2), turned to 90 degrees
- moved R7 1.05 mm to (146.2, 103.2)
Connections:
- J1 pad 0: GND -> AGND
- J1 pad 10: GND -> AGND
- J1 pad 17: GND -> AGND
- J1 pad 18: GND -> AGND
- J1 pad 21: GND -> AGND
- J1 pad 22: GND -> AGND
- J1 pad 3: GND -> AGND
- J1 pad 5: GND -> AGND
- J1 pad 7: GND -> AGND
- Q1 pad 2: GND -> AGND
- Q2 pad 2: GND -> AGND
- Q3 pad 2: GND -> AGND
- Q4 pad 2: GND -> AGND
- R1 pad 2: GND -> AGND
- R2 pad 2: GND -> AGND
- R3 pad 2: GND -> AGND
- R9 pad 2: GND -> AGND
- RV1 pad 3: GND -> AGND
- RV2 pad 3: GND -> AGND
- SW1 pad 1: GND -> AGND
- U1 pad 13: GND -> AGND
- U1 pad 16: Net-(U1-GP12) -> unconnected-(U1-GP12-Pad16)
- U1 pad 18: GND -> AGND
- U1 pad 23: GND -> AGND
- U1 pad 28: GND -> AGND
- U1 pad 3: GND -> AGND
- U1 pad 33: GND -> AGND
- U1 pad 34: unconnected-(U1-GP28-Pad34) -> Net-(U1-GP28)
- U1 pad 38: GND -> AGND
- U1 pad 8: GND -> AGND
- U2 pad 1: Net-(U1-GP12) -> Net-(U1-GP28)
- U2 pad 11: GND -> AGND
- U2 pad 16: GND -> AGND
- U2 pad 3: Net-(U1-3V3_EN) -> Net-(U2-~{RESET})
- U3 pad 1: (no net) -> unconnected-(U3-N_C-Pad1)
- U3 pad 2: (no net) -> AGND
- U3 pad 3: (no net) -> +5V
- U3 pad 4: GND -> +5V
- U3 pad 5: (no net) -> +2V5REF
- U4 pad 2: GND -> AGND
Routing:
- net Net-(U2-~{RESET}): track 0.00 -> 35.9 mm, vias 0 -> 2
- net Net-(U1-GP12): track 32.4 -> 0.00 mm, vias 2 -> 0
- net GND: track 32.2 -> 0.00 mm, vias 8 -> 0
- net AGND: track 65.1 -> 45.6 mm, vias 3 -> 9
- net +2V5REF: track 52.1 -> 66.0 mm, vias 2 -> 3
- net Net-(U1-3V3_EN): track 31.0 -> 17.5 mm, vias 2 -> 1
- net Net-(U1-GP28): track 0.00 -> 9.25 mm, vias 0 -> 1
- net Net-(J1-P19): track 54.8 -> 55.9 mm
- net +12V: track 59.5 -> 60.6 mm, vias 3 -> 1
- net Net-(U2-VOUT): track 72.9 -> 73.5 mm
- added copper zone on B.Cu, net AGND
- removed copper zone on B.Cu, net GND

Commit message: PCD 1st version
Parts:
- removed C1, C2: 4.7 µF, Capacitor_SMD:C_0402_1005Metric_Pad0.74x0.62mm_HandSolder
- removed G*** (x2): LOGO, UW-Madison Logo:logo
- added C_in: 22 µF, Capacitor_SMD:C_1206_3216Metric_Pad1.33x1.80mm_HandSolder, F.Cu at (120.0, 102.5)
- added C_out: 22 µF, Capacitor_SMD:C_1206_3216Metric_Pad1.33x1.80mm_HandSolder, F.Cu at (112.5, 102.5)
- SW1, SW2: value SW_Push -> 3-1825910-5; footprint Button_Switch_SMD:SW_Tactile_SPST_NO_Straight_CK_PTS636Sx25SMTRLFS -> TE_3_1825910_5:SW4_1825910-I_TEC
- U1: value SC0915 -> Raspberry Pi Pico
- U3: value LM4132BMF-2.5 -> LM4132BMF-2.5/NOPB
- moved SW2 62.6 mm to (120.8, 78.8), turned to 0 degrees
- moved U3 51.2 mm to (115.0, 97.0), turned to 0 degrees
- moved U2 47.0 mm to (115.0, 120.0)
- moved R10 20.1 mm to (120.8, 113.5)
- moved SW1 7.00 mm to (167.8, 117.7), turned to 180 degrees
- moved Q1 0.80 mm to (169.0, 75.8)
- moved Q2 0.80 mm to (158.5, 75.8)
- moved Q3 0.80 mm to (148.0, 75.8)
- moved Q4 0.80 mm to (137.5, 75.8)
- moved R1 0.80 mm to (174.0, 75.8)
- moved R2 0.80 mm to (163.5, 75.8)
- moved R3 0.80 mm to (153.0, 75.8)
- moved R4 0.80 mm to (169.5, 80.8)
- moved R5 0.80 mm to (159.0, 80.8)
- moved R6 0.80 mm to (148.5, 80.8)
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Connections:
- SW1 pad 2: Net-(U1-3V3_EN) -> AGND
- SW2 pad 1: Net-(U2-~{RESET}) -> AGND
Routing:
- net Net-(U1-GP5): track 6.73 -> 60.1 mm, vias 0 -> 2
- net Net-(U1-GP4): track 6.97 -> 58.7 mm, vias 0 -> 2
- net Net-(U1-GP6): track 7.14 -> 56.9 mm, vias 0 -> 2
- net Net-(U1-GP28): track 9.25 -> 57.8 mm
- net Net-(U2-~{RESET}): track 35.9 -> 80.7 mm, vias 2 -> 3
- net Net-(U1-GP7): track 11.4 -> 55.3 mm, vias 1 -> 2
- net +12V: track 60.6 -> 36.0 mm
- net Net-(U2-VOUT): track 73.5 -> 51.1 mm
- net AGND: track 45.6 -> 34.6 mm
- net +2V5REF: track 66.0 -> 71.5 mm, vias 3 -> 7
- net Net-(Q2-G): track 26.6 -> 21.4 mm, vias 2 -> 1
- net Net-(Q4-G): track 42.6 -> 39.9 mm, vias 2 -> 1
- net Net-(J1-P19): track 55.9 -> 58.3 mm
- net Net-(U1-GP26): track 73.5 -> 71.7 mm
- net Net-(U1-3V3_EN): track 17.5 -> 15.9 mm, vias 1 -> 0
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Other:
- board text added: "SWCLK"
- board text added: "SWDIO"

Commit message: update
Routing:
- net AGND: track 34.6 -> 36.8 mm
