File: control_board_Kicad/KiCad-Pi-Pico/KiCad-Pi-Pico.kicad_sch (KiCad schematic)
At the start: 21 parts, among them J1 DB25_Plug_MountingHoles, Q1 2N7000, Q2 2N7000, Q3 2N7000, Q4 2N7000, SW1 SW_Push, U1 SC0915, U2 AD5761RBRUZ

Commit message: update KiCad design
Parts:
- removed Q1, Q2, Q3, Q4: 2N7000, Package_TO_SOT_THT:TO-92_Inline, symbol Transistor_FET:2N7000
- removed RN1, RN2, RN3, RN4: VoltageDivider, symbol Device:VoltageDivider
- added Q1, Q2, Q3, Q4: 2N7002, Package_TO_SOT_SMD:SOT-23, symbol Transistor_FET:2N7002
- added R10, R11, R12, R13, R14: 4.7 kΩ, Resistor_SMD:R_1206_3216Metric_Pad1.30x1.75mm_HandSolder, symbol Device:R_US
- added RV1, RV2: R_Potentiometer_US, Potentiometer_THT:Potentiometer_Bourns_3386W_Horizontal, symbol Device:R_Potentiometer_US
- added U3: LM285D-2.5, Package_SO:SOIC-8_3.9x4.9mm_P1.27mm, symbol Reference_Voltage:LM285D-2.5
- R1, R2, R3, R4, R5, R6, R7, R8, R9: value R_US -> 4.7 kΩ; footprint (none) -> Resistor_SMD:R_1206_3216Metric_Pad1.30x1.75mm_HandSolder
- SW1: footprint (none) -> Button_Switch_SMD:SW_Tactile_SPST_NO_Straight_CK_PTS636Sx25SMTRLFS
Connections:
- net +3.3VADC: now also RV1.2
- net +5V: now also R10.1, R11.1, R12.1, R13.1, R14.1
- net +5VREF: now also RV1.1
- net GND: now also U2.5 (AGND), U2.6 (VSS), Q1.2 (S), Q2.2 (S), Q3.2 (S), Q4.2 (S), RV1.3, RV2.3, U3.4 (A)
- net at J1.9, R8.2: now also Q4.3 (D)
- net at J1.16 (P16), R5.2: now also Q2.3 (D)
- net at R3.1, U1.11 (GP8): now also Q3.1 (G)
- net at J1.20 (P20), R6.2: now also Q3.3 (D)
- net at R2.1, U1.2 (GP1): now also Q2.1 (G)
- net at U1.31 (GP26): now also RV2.2
- net at R1.1, U1.1 (GP0): now also Q1.1 (G)
- net at J1.14 (P14): now also RV2.1
- net at J1.8, U1.12 (GP9): now also R13.2
- net at J1.23 (P23), U1.14 (GP10): now also R12.2
- net at J1.24 (P24), U1.15 (GP11): now also R11.2
- net at R9.1, U1.4 (GP2): now also Q4.1 (G)
- net at J1.6, U1.5 (GP3): now also R14.2
- net at J1.15 (P15), R4.2: now also Q1.3 (D)
- net +2V5 renamed +2V5REF
- net +2V5REF: now also R10.2, U3.8 (K)
Other:
- note added: "2.5V voltage reference"
- note added: "2N7002"
- note added: "ALL RESISTORS 1206 FOOTPRINT"
- note added: "Local/Remote(Output)(M)"
- note added: "Pending voltage booster"
- note removed: "(0–5V)"
- note removed: "2.5V reference by voltage divider"
- note removed: "How to generate this 10V? VDD must be decoupled to AGND."
- note removed: "Please check if my spi interface is correctly connected."
- note removed: "Separate ground?"
- note removed: "Step down to 0-2.5V and use the pico ADC"
- note removed: "Vss should be grounded, must be decoupled to AGND."
- note removed: "What's the difference between Reference & common??? They use one reference for Start/Stop, CW/CCW, and Prime. But four separate common for one function? The spec mention the following: Motor running relay (Closed when running, 1 A max @ 24 VDC) General alarm relay (Closed when error is displayed, 1 A @ 24 VDC) Open head relay (Closed when activated, 1 A @ 24 VDC)"
- note removed: "voltage divider for 2.5V reference"

Commit message: KiCad update
Connections:
- net +5VREF is gone; now on net +5V: RV1.1
