File: control_board_Kicad/KiCad-Pi-Pico/KiCad-Pi-Pico.kicad_sch (KiCad schematic)
At the start: 25 parts, among them J1 DB25_Plug_MountingHoles, Q1 2N7002, Q2 2N7002, Q3 2N7002, Q4 2N7002, SW1 SW_Push, U1 SC0915, U2 AD5761RBRUZ, U3 LM285D-2.5

Commit message: KiCad updated
Parts:
- U1: footprint SC0915:MODULE_SC0915 -> RPi_Pico:RPi_Pico_SMD_TH
Changed lines of the file:
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@@
 			)
 		)
-		(property "Footprint" "SC0915:MODULE_SC0915"
+		(property "Footprint" "RPi_Pico:RPi_Pico_SMD_TH"
 			(at 177.8 74.93 0)
 			(effects

Commit message: PCB design finished
Parts:
- added U4: PCN2-S5-S12-S, PCN2_S5_S12_S:CONV_PCN2-S5-S12-S, symbol PCN2-S5-S12-S:PCN2-S5-S12-S
Connections:
- net +5V: now also U4.1 (+VIN)
- net GND: now also J1.0 (PAD), U4.2 (-VIN); no longer U2.5 (AGND), U2.6 (VSS)
- net +10V renamed +12V
- net +12V: now also U4.6 (+VOUT)
- new net AGND: U2.5 (AGND), U2.6 (VSS), U4.4 (-VOUT)
Other:
- note removed: "Pending voltage booster"

Commit message: update
Parts:
- removed U3: LM285D-2.5, Package_SO:SOIC-8_3.9x4.9mm_P1.27mm, symbol Reference_Voltage:LM285D-2.5
- added C1, C2: C_Small, symbol Device:C_Small
- added SW2: SW_Push, symbol Switch:SW_Push
- added U3: LM4132BMF-2.5/NOPB, LM4132BMF_2_5_NOPB:DBV0005A_M, symbol LM4132BMF_2_5_NOPB:LM4132BMF-2.5_NOPB
- added U5: LM285LPR-2-5, LM285LPR_2_5:LP3, symbol LM285LPR_2_5:LM285LPR-2-5
- U1: footprint RPi_Pico:RPi_Pico_SMD_TH -> SC0915:MODULE_SC0915
- U4: footprint PCN2_S5_S12_S:CONV_PCN2-S5-S12-S -> CONV_PCN2-S5-S12-S
Connections:
- net GND is gone; now on net AGND: J1.0 (PAD), J1.10, J1.17 (P17), J1.18 (P18), J1.21 (P21), J1.22 (P22), J1.3, J1.5, J1.7, Q1.2 (S), Q2.2 (S), Q3.2 (S), Q4.2 (S), R1.2, R2.2, R3.2, R9.2, RV1.3, RV2.3, SW1.1, U1.13 (GND), U1.18 (GND), U1.23 (GND), U1.28 (GND), U1.3 (GND), U1.33 (AGND), U1.38 (GND), U1.8 (GND), U1.A (USB_SHIELD), U1.B (USB_SHIELD), U1.C (USB_SHIELD), U1.D (USB_SHIELD), U1.D2 (GND), U2.11 (~{LDAC}), U2.16 (DGND), U4.2 (-VIN)
- net +2V5REF: now also C2.2, U3.5 (VREF), U5.2 (CATHODE)
- net +5V: now also C1.2, U3.3 (EN), U3.4 (VIN)
- net AGND: now also C1.1, C2.1, SW2.2, U3.2 (GND), U5.1 (ANODE)
- net at U1.16 (GP12): no longer U2.1 (~{ALERT})
- net at U1.34 (GP28): now also U2.1 (~{ALERT})
- net at SW1.2, U1.37 (3V3_EN): no longer U2.3 (~{RESET})
- new net: SW2.1, U2.3 (~{RESET})
- no-connect marks 14 -> 26
Other:
- note added: "Hard reset button(DAC)"
- note added: "Hard reset button(pico)"
- note removed: "3.3V output convert by the Pico"
- note removed: "Hard reset button(tie to both pico and the DAC)"
- note removed: "Main power input, pico can take 1.8V to 5.5V"
- moved on the sheet: R10, RV1, SW1, U4

Commit message: update PCB design
Parts:
- C1, C2: value C_Small -> 4.7 µF; footprint (none) -> Capacitor_SMD:C_0402_1005Metric_Pad0.74x0.62mm_HandSolder
- SW2: footprint (none) -> Button_Switch_SMD:SW_Tactile_SPST_NO_Straight_CK_PTS636Sx25SMTRLFS
- U1: value SC0915 -> Raspberry Pi Pico
Other:
- company: UW-Madison -> UW-Madison Chemistry Department Stahl Group
Changed lines of the file:
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@@
 	(title_block
 		(title "Pi Pico Masterflex pump DB25 control board")
-		(date "2024-07-22")
-		(rev "0.1")
-		(company "UW-Madison")
+		(date "2024-09-25")
+		(rev "1.0")
+		(company "UW-Madison Chemistry Department Stahl Group")
+		(comment 1 "Made by Tom Tan")
 	)
 	(junction
@@
 			)
 		)
-		(property "Footprint" ""
+		(property "Footprint" "Button_Switch_SMD:SW_Tactile_SPST_NO_Straight_CK_PTS636Sx25SMTRLFS"
 			(at 119.38 80.01 0)
 			(effects
@@
 			)
 		)
-		(property "Value" "C_Small"
+		(property "Value" "4.7 µF"
 			(at 326.39 99.0535 0)
 			(effects
@@
 			)
 		)
-		(property "Footprint" ""
+		(property "Footprint" "Capacitor_SMD:C_0402_1005Metric_Pad0.74x0.62mm_HandSolder"
 			(at 323.85 97.79 0)
 			(effects
@@
 			)
 		)
-		(property "Value" "C_Small"
+		(property "Value" "4.7 µF"
 			(at 326.39 81.2862 0)
 			(effects
@@
 			)
 		)
-		(property "Footprint" ""
+		(property "Footprint" "Capacitor_SMD:C_0402_1005Metric_Pad0.74x0.62mm_HandSolder"
 			(at 323.85 80.01 0)
 			(effects
@@
 					(size 1.27 1.27)
 				)
+				(hide yes)
 			)
 		)
-		(property "Value" "SC0915"
+		(property "Value" "Raspberry Pi Pico"
 			(at 177.8 29.21 0)
 			(effects

Commit message: PCD 1st version
Parts:
- removed SW1, SW2: SW_Push, Button_Switch_SMD:SW_Tactile_SPST_NO_Straight_CK_PTS636Sx25SMTRLFS, symbol Switch:SW_Push
- added SW1, SW2: 3-1825910-5, SW4_1825910-I_TEC, symbol TE_3_1825910_5:3-1825910-5
- C1, C2: value 4.7 µF -> 22 µF; footprint Capacitor_SMD:C_0402_1005Metric_Pad0.74x0.62mm_HandSolder -> Capacitor_SMD:C_1206_3216Metric_Pad1.33x1.80mm_HandSolder
Connections:
- net AGND: now also SW1.1, SW1.2, SW2.1, SW2.2
- net at U2.3 (~{RESET}): now also SW2.3, SW2.4
- net at U1.37 (3V3_EN): now also SW1.3, SW1.4
- no-connect marks 26 -> 28
Other:
- note removed: "Both debug pin"
- note removed: "Hard reset button(DAC)"
