File: control_board_Kicad/potentiostat control/potentiostat control.kicad_sch (KiCad schematic)
At the start: 8 parts, among them J1 L717SDA15PA4CH4F, Q1 2N7002, Q2 2N7002, SW1 3-1825910-5, U1 Raspberry Pi Pico

Commit message: update board
Parts:
- removed J1: L717SDA15PA4CH4F, CONN_L717SDA15PA4CH4F_AMP, symbol DB15:L717SDA15PA4CH4F
- added J1: L717HDE15PD1CH4F, DB15_L717HDE15PD1CH4F:AMPHENOL_L717HDE15PD1CH4F, symbol DB15_L717HDE15PD1CH4F:L717HDE15PD1CH4F
Connections:
- net DGND is gone; now on net GND: Q2.2 (S)
- net +5VP: now also J1.15
- net AGND: now also J1.2
- net GND: now also J1.6
- net at U1.34 (GP28): now also J1.1
- net at U1.12 (GP9): now also J1.10
- net at Q2.3 (D), R3.2: now also J1.11, J1.12, J1.13, J1.14
- net at U1.9 (GP6): now also J1.7
- net at U1.10 (GP7): now also J1.8
- net at U1.11 (GP8): now also J1.9
- new net: J1.SH1 (SHIELD), J1.SH2 (SHIELD)
- no-connect marks 31 -> 32
Other:
- moved on the sheet: R2
